File: pcb/dev board.kicad_pcb (KiCad board)
At the start: 2 copper layers, 21 x 51.2 mm, 35 parts, among them J1 USB_C_Receptacle_USB2.0_14P, J2 Conn_01x20, J3 Conn_01x03, J5 Conn_01x20, SW1 SW_Push, U1 RP2040, U2 NCP1117-3.3_SOT223, U4 W25Q16JVUXIQ TR, Y1 12 MHz

Commit message: Update PCB files
Parts:
- added C18: 10u, Capacitor_SMD:C_0603_1608Metric, F.Cu at (122.5, 116.8)
- added C19: 0.1uf, Capacitor_SMD:C_0402_1005Metric, F.Cu at (128.5, 118.0)
- added J4: 104031-0811, Connector_Card:microSD_HC_Molex_104031-0811, B.Cu at (124.4, 115.2)
- added R10: 10k, Resistor_SMD:R_0402_1005Metric, F.Cu at (126.0, 116.0)
- added R8: 10k, Resistor_SMD:R_0402_1005Metric, F.Cu at (127.2, 112.2)
- added R9: 10k, Resistor_SMD:R_0402_1005Metric, F.Cu at (119.5, 117.0)
- G***: moved to B.Cu
- J3: footprint Connector_PinHeader_2.54mm:PinHeader_1x03_P2.54mm_Vertical -> Connector_PinHeader_1.27mm:PinHeader_1x03_P1.27mm_Vertical_SMD_Pin1Left
- moved G*** 15.4 mm to (118.5, 101.5), turned to -90 degrees
- moved G*** 10.0 mm to (126.8, 96.5)
- moved J3 3.29 mm to (123.2, 120.5), turned to 180 degrees
- moved J2 3.25 mm to (135.0, 73.6)
- moved C12 0.50 mm to (127.0, 106.5), turned to 45 degrees
- moved R5 0.35 mm to (123.0, 107.0)
Connections:
- J2 pad 16: GPIO19 -> unconnected-(J2-Pin_16-Pad16)
- J2 pad 17: GPIO18 -> unconnected-(J2-Pin_17-Pad17)
- J2 pad 19: GPIO17 -> unconnected-(J2-Pin_19-Pad19)
- J2 pad 20: GPIO16 -> unconnected-(J2-Pin_20-Pad20)
- U1 pad 27: GPIO16 -> SD_MISO
- U1 pad 28: GPIO17 -> SD_CS
- U1 pad 29: GPIO18 -> SD_SCK
- U1 pad 30: GPIO19 -> SD_MOSI
Routing:
- net +3V3: track 101.5 -> 169.6 mm, vias 8 -> 10
- net GND: track 93.3 -> 139.3 mm, vias 7 -> 21
- net SD_MOSI: track 0.00 -> 39.3 mm, vias 0 -> 4
- net SD_SCK: track 0.00 -> 29.0 mm, vias 0 -> 6
- net SD_CS: track 0.00 -> 22.4 mm, vias 0 -> 3
- net GPIO16: track 21.3 -> 0.00 mm, vias 1 -> 0
- net GPIO17: track 19.1 -> 0.00 mm, vias 1 -> 0
- net SD_MISO: track 0.00 -> 18.1 mm, vias 0 -> 2
- net SWDIO: track 20.4 -> 34.3 mm, vias 1 -> 4
- net GPIO18: track 13.5 -> 0.00 mm, vias 1 -> 0
- net GPIO19: track 11.7 -> 0.00 mm, vias 1 -> 0
- net SWCLK: track 22.8 -> 28.7 mm, vias 1 -> 2
- net GPIO20: track 11.1 -> 14.6 mm
- net GPIO22: track 6.69 -> 10.2 mm
- net VBUS: track 23.9 -> 27.4 mm
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Other:
- board size 21 x 51.2 mm -> 24.2 x 51.2 mm
- copper layers 2 -> 4
