File: pcb/dev board.kicad_sch (KiCad schematic)
At the start: 33 parts, among them J1 USB_C_Receptacle_USB2.0_14P, J2 Conn_01x20, J3 Conn_01x03, J5 Conn_01x20, SW1 SW_Push, U1 RP2040, U2 NCP1117-3.3_SOT223, U4 W25Q16JVUXIQ TR, Y1 12 MHz

Commit message: Update PCB files
Parts:
- added C18: 10u, Capacitor_SMD:C_0603_1608Metric, symbol Device:C
- added C19: 0.1uf, Capacitor_SMD:C_0402_1005Metric, symbol Device:C
- added J4: 104031-0811, Connector_Card:microSD_HC_Molex_104031-0811, symbol sd card123:104031-0811
- added R10, R8, R9: 10k, Resistor_SMD:R_0402_1005Metric, symbol Device:R
- J3: footprint Connector_PinHeader_2.54mm:PinHeader_1x03_P2.54mm_Vertical -> Connector_PinHeader_1.27mm:PinHeader_1x03_P1.27mm_Vertical_SMD_Pin1Left
Connections:
- net +3V3: now also C18.1, C19.2, J4.4 (VDD), R10.1, R8.1, R9.1
- net GND: now also C18.2, C19.1, J4.6 (VSS), J4.G1 (GND), J4.G2 (GND), J4.G3 (GND), J4.G4 (GND)
- net GPIO16: no longer names the net of J2.20 (Pin_20)
- net GPIO16: no longer U1.27 (GPIO16)
- net GPIO17: no longer names the net of J2.19 (Pin_19)
- net GPIO17: no longer U1.28 (GPIO17)
- net GPIO18: no longer names the net of J2.17 (Pin_17)
- net GPIO18: no longer U1.29 (GPIO18)
- net GPIO19: no longer names the net of J2.16 (Pin_16)
- net GPIO19: no longer U1.30 (GPIO19)
- new net SD_CS: J4.2 (CD/DAT3), R8.2, U1.28 (GPIO17)
- new net SD_MISO: J4.7 (DAT0), R9.2, U1.27 (GPIO16)
- new net SD_MOSI: J4.3 (CMD), R10.2, U1.30 (GPIO19)
- new net SD_SCK: J4.5 (CLK), U1.29 (GPIO18)
- no-connect marks 0 -> 12
Other:
- note added: "sd card"
- moved on the sheet: C15, C16, C17, R5, R6, R7, SW1, U4, Y1
